Commit message: Lidar in Ridgeback

File: rbkk3-ros2ws/src/ridgeback_description/urdf/accessories.urdf.xacro (robot description, xacro)
@@ -9,14 +9,17 @@
     ridgeback_base/launch/base.launch
   -->
-  <!-- sick_lms1xx commented out for the moment -->
+  <!-- Only leaving Hokuyo LIDAR -->
   <!--xacro:include filename="$(find ridgeback_description)/urdf/accessories/sick_lms1xx_mount.urdf.xacro" /-->
   <!--xacro:include filename="$(find ridgeback_description)/urdf/accessories/sick_s300_mount.urdf.xacro" /-->
   <xacro:include filename="$(find ridgeback_description)/urdf/accessories/hokuyo_ust-10lx_mount.urdf.xacro" />
-  <!-- If enabled, generate the front HOKUYO UST-10LX LASER payload. -->
-  <xacro:if value="$(optenv RIDGEBACK_FRONT_HOKUYO_LASER 0)">
-    <xacro:hokuyo_ust-10lx_mount prefix="front"
-                                 topic="front/scan"
-                                 location="1" />
-  </xacro:if>
+  <!-- Force generate the front HOKUYO UST-10LX LASER payload. -->
+  <!--xacro:if value="$(optenv RIDGEBACK_FRONT_HOKUYO_LASER 0)"-->
+  <xacro:hokuyo_ust-10lx_mount  prefix="front"
+                                topic="front/scan"
+                                location="1"
+                                sim_ignition="true"
+                                tf_prefix="$(arg name)/"
+                                 />
+  <!--/xacro:if-->
   <!-- If enabled, generate the rear HOKUYO UST-10LX LASER payload. -->
   <xacro:if value="$(optenv RIDGEBACK_REAR_HOKUYO_LASER 0)">

File: rbkk3-ros2ws/src/ridgeback_description/urdf/accessories/hokuyo_ust-10lx_mount.urdf.xacro (robot description, xacro)
@@ -1,5 +1,5 @@
 <?xml version="1.0"?>
 <robot xmlns:xacro="http://ros.org/wiki/xacro">
-  <xacro:macro name="hokuyo_ust-10lx_mount" params="prefix topic location">
+  <xacro:macro name="hokuyo_ust-10lx_mount" params="prefix topic location sim_ignition:=false tf_prefix:=rbkk3/">
     <joint name="${prefix}_laser_joint" type="fixed">
       <origin xyz="${location * 0.3932} 0 0.2330" rpy="0 0 ${PI/2 - (location * PI/2)}" />
@@ -30,38 +30,36 @@
       </collision>
     </link>
-    <gazebo reference="${prefix}_laser">
-      <turnGravityOff>false</turnGravityOff>
-      <sensor type="ray" name="${prefix}_laser">
-        <pose>0 0 0 0 0 0</pose>
-        <visualize>false</visualize>
-        <update_rate>50</update_rate>
-        <ray>
-          <scan>
-            <horizontal>
-              <samples>720</samples>
-              <resolution>1</resolution>
-              <min_angle>-2.35619</min_angle>
-              <max_angle>2.35619</max_angle>
-            </horizontal>
-          </scan>
-          <range>
-            <min>0.20</min>
-            <max>10.0</max>
-            <resolution>0.01</resolution>
-          </range>
-          <noise>
-            <type>gaussian</type>
-            <mean>0.0</mean>
-            <stddev>0.001</stddev>
-          </noise>
-        </ray>
-        <plugin name="gazebo_ros_laser" filename="libgazebo_ros_laser.so">
-          <topicName>${topic}</topicName>
-          <frameName>${prefix}_laser</frameName>
-          <hokuyoMinIntensity>101</hokuyoMinIntensity>
-        </plugin>
-      </sensor>
-      <material>Gazebo/DarkGrey</material>
-    </gazebo>
+    <!-- Ignition reference -->
+    <xacro:if value="${sim_ignition}">
+      <gazebo reference="${prefix}_laser">
+        <sensor name="${prefix}_laser_sensor" type="gpu_lidar">
+          <update_rate>50</update_rate>
+          <visualize>true</visualize>
+          <always_on>true</always_on>
+          <ignition_frame_id>${tf_prefix}${prefix}_laser</ignition_frame_id>
+          <lidar>
+            <scan>
+              <horizontal>
+                <samples>720</samples>
+                <resolution>1</resolution>
+                <min_angle>-2.35619</min_angle>
+                <max_angle>2.35619</max_angle>
+              </horizontal>
+              <vertical>
+                <samples>1</samples>
+                <resolution>1</resolution>
+                <min_angle>0</min_angle>
+                <max_angle>0</max_angle>
+              </vertical>
+            </scan>
+            <range>
+              <min>0.20</min>
+              <max>10</max>
+              <resolution>0.01</resolution>
+            </range>
+          </lidar>
+        </sensor>
+      </gazebo>
+    </xacro:if>
   </xacro:macro>
 </robot>
