Commit message: cleaned up data files interactions and now using effort interfaces

File: rbkk3-ros2ws/src/rbkk3_description/urdf/rbkk3.xacro (robot description, xacro)
@@ -2,13 +2,25 @@
 <robot xmlns:xacro="http://www.ros.org/wiki/xacro" name="rbkk3">
     <xacro:arg name="name" default="rbkk3"/>
+    <xacro:arg name="use_prefix" default="true"/>
+    <!--xacro:arg name="namespace" default="/"/-->
+    <xacro:if value="$(arg use_prefix)">
+        <xacro:property name="prefix" value="$(arg name)/"/>
+        <xacro:property name="cm_namespace" value="$(arg name)"/>
+    </xacro:if>
+    <xacro:unless value="$(arg use_prefix)">
+        <xacro:property name="prefix" value=""/>
+        <xacro:property name="cm_namespace" value="/"/>
+    </xacro:unless>
     <xacro:arg name="sim_ignition" default="false" />
-    <xacro:arg name="simulation_controllers" default="$(find rbkk3_description)/config/rbkk3_controllers.yaml" />
+    <xacro:arg name="simulation_controllers" default="$(find rbkk3_description)/config/$(arg name)_controllers.yaml" />
     <!-- Platform -->
-    <xacro:include filename="$(find ridgeback_description)/urdf/ridgeback.urdf.xacro" ns="rb"/>
+    <xacro:arg name="platform_prefix" default="platform/"/>
+    <xacro:include filename="$(find ridgeback_description)/urdf/ridgeback_model.xacro" ns="rb"/>
+    <xacro:rb.load_platform prefix="${prefix}$(arg platform_prefix)" sim_ignition="$(arg sim_ignition)"/>
     <!-- Arm -->
     <xacro:arg name="arm_prefix" default="arm/"/>
-    <xacro:include filename="$(find rbkk3_description)/urdf/rbkk3_arm.urdf.xacro" ns="kk"/>
+    <xacro:include filename="$(find rbkk3_description)/urdf/rbkk3_arm.xacro" ns="kk"/>
     <xacro:kk.load_robot
-        parent="rbkk3_integration_link"
+        parent="${prefix}rbkk3_integration_link"
         arm="$(arg arm)"
         gripper="$(arg gripper)"
@@ -26,5 +38,5 @@
         connection_inactivity_timeout_ms="$(arg connection_inactivity_timeout_ms)"
         use_internal_bus_gripper_comm="$(arg use_internal_bus_gripper_comm)"
-        prefix="$(arg arm_prefix)"
+        prefix="${prefix}$(arg arm_prefix)"
         use_fake_hardware="$(arg use_fake_hardware)"
         fake_sensor_commands="$(arg fake_sensor_commands)"
@@ -36,5 +48,5 @@
     </xacro:kk.load_robot>
     <!-- Integration Plate -->
-    <link name="rbkk3_integration_link">
+    <link name="${prefix}rbkk3_integration_link">
         <visual>
         <origin xyz="0 0 0" rpy="0 0 0" />
@@ -45,8 +57,8 @@
       </visual>
     </link>
-    <joint name="rbkk3_integration_platform_joint" type="fixed">
+    <joint name="${prefix}rbkk3_integration_platform_joint" type="fixed">
         <origin xyz="0.25 0 0.0" rpy="0 0 0"/>
-        <parent link="mid_mount"/>
-        <child link="rbkk3_integration_link"/>
+        <parent link="${prefix}$(arg platform_prefix)mid_mount"/>
+        <child link="${prefix}rbkk3_integration_link"/>
     </joint>
     <!-- Controller Manager Spawner for Ignition -->
@@ -56,5 +68,5 @@
                 <parameters>$(arg simulation_controllers)</parameters>
                 <ros>
-                    <namespace>$(arg namespace)</namespace>
+                    <namespace>${cm_namespace}</namespace>
                 </ros>
             </plugin>

File: rbkk3-ros2ws/src/ridgeback_description/urdf/accessories.urdf.xacro (robot description, xacro)
@@ -15,9 +15,9 @@
   <!-- Force generate the front HOKUYO UST-10LX LASER payload. -->
   <!--xacro:if value="$(optenv RIDGEBACK_FRONT_HOKUYO_LASER 0)"-->
-  <xacro:hokuyo_ust-10lx_mount  prefix="front"
+  <xacro:hokuyo_ust-10lx_mount  prefix="${prefix}"
+                                laser_prefix="front"
                                 topic="front/scan"
                                 location="1"
-                                sim_ignition="true"
-                                tf_prefix="$(arg name)/"
+                                sim_ignition="${sim_ignition}"
                                  />
   <!--/xacro:if-->

File: rbkk3-ros2ws/src/ridgeback_description/urdf/accessories/hokuyo_ust-10lx_mount.urdf.xacro (robot description, xacro)
@@ -1,11 +1,11 @@
 <?xml version="1.0"?>
 <robot xmlns:xacro="http://ros.org/wiki/xacro">
-  <xacro:macro name="hokuyo_ust-10lx_mount" params="prefix topic location sim_ignition:=false tf_prefix:=rbkk3/">
-    <joint name="${prefix}_laser_joint" type="fixed">
+  <xacro:macro name="hokuyo_ust-10lx_mount" params="prefix:='' laser_prefix topic location sim_ignition:=false/">
+    <joint name="${prefix}${laser_prefix}_laser_joint" type="fixed">
       <origin xyz="${location * 0.3932} 0 0.2330" rpy="0 0 ${PI/2 - (location * PI/2)}" />
-      <parent link="chassis_link" />
-      <child link="${prefix}_laser" />
+      <parent link="${prefix}chassis_link" />
+      <child link="${prefix}${laser_prefix}_laser" />
     </joint>
-    <link name="${prefix}_laser">
+    <link name="${prefix}${laser_prefix}_laser">
       <inertial>
         <mass value="0.130" />
@@ -32,10 +32,10 @@
     <!-- Ignition reference -->
     <xacro:if value="${sim_ignition}">
-      <gazebo reference="${prefix}_laser">
-        <sensor name="${prefix}_laser_sensor" type="gpu_lidar">
+      <gazebo reference="${prefix}${laser_prefix}_laser">
+        <sensor name="${prefix}${laser_prefix}_laser_sensor" type="gpu_lidar">
           <update_rate>50</update_rate>
           <visualize>true</visualize>
           <always_on>true</always_on>
-          <ignition_frame_id>${tf_prefix}${prefix}_laser</ignition_frame_id>
+          <ignition_frame_id>${prefix}${laser_prefix}_laser</ignition_frame_id>
           <lidar>
             <scan>
